File: ThumbsUp.kicad_pcb (KiCad board)
At the start: 2 copper layers, 251.1 x 336.1 mm, 150 parts, among them IC1 RP2040, IC2 W25Q128JVSIM, J1 Conn_01x04_Male, J10 Raiser_Male, J11 Raiser_Female, J12 Raiser_Male, J13 Raiser_Female, J14 Raiser_Male, J15 Raiser_Female, J16 Raiser_Male, J17 Raiser_Female, J18 Raiser_Male, J19 52559-1233, J2 Conn_01x04_Male, J20 Conn_01x04_Female, J21 Conn_01x04_Female, J22 Conn_01x04_Female, J23 Conn_01x04_Female, J24 Conn_01x04_Male, J25 Conn_01x04_Male, J26 Conn_01x04_Male, J27 Conn_01x04_Male, J28 Conn_01x04_Female, J29 Conn_01x04_Female, J3 Conn_01x04_Female, J30 Conn_01x04_Female, J31 Conn_01x04_Female, J4 Conn_01x04_Male, J5 Conn_01x04_Female, J6 Conn_01x04_Male, J7 Conn_01x04_Male, J8 Conn_01x04_Male, J9 Raiser_Female, U1 NCP1117-3.3_SOT223, Y1 ABLS-12.000MHZ-B4-T

Commit message: Wiring continued
Parts:
- moved C7 1.41 mm to (154.8, 220.0)
- moved C6 1.28 mm to (139.7, 219.8)
- moved C1 1.14 mm to (139.6, 209.8)
- moved C3 0.88 mm to (139.6, 212.1)
- moved C10 0.62 mm to (139.7, 214.4)
Connections:
- IC1 pad 2: Net-(IC1-Pad2) -> ROW0
- IC1 pad 3: Net-(IC1-Pad3) -> ROW1
- IC1 pad 34: Net-(IC1-Pad34) -> COL4
- IC1 pad 35: Net-(IC1-Pad35) -> COL0
- IC1 pad 36: Net-(IC1-Pad36) -> COL1
- IC1 pad 37: Net-(IC1-Pad37) -> COL2
- IC1 pad 38: Net-(IC1-Pad38) -> COL3
- IC1 pad 39: Net-(IC1-Pad39) -> COL5
- IC1 pad 4: Net-(IC1-Pad4) -> COL7
- IC1 pad 40: Net-(IC1-Pad40) -> ROW3
- IC1 pad 41: Net-(IC1-Pad41) -> ROW2
- IC1 pad 5: Net-(IC1-Pad5) -> COL6
- IC1 pad 6: Net-(IC1-Pad6) -> COL8
- IC1 pad 7: Net-(IC1-Pad7) -> COL9
- IC1 pad 8: Net-(IC1-Pad8) -> COLA
- IC1 pad 9: Net-(IC1-Pad9) -> COLB
Routing:
- net ROW3: track 15.7 -> 154.5 mm
- net ROW2: track 27.0 -> 120.1 mm
- net Net-(BOOTSEL1-Pad1): track 3.60 -> 61.4 mm, vias 0 -> 2
- net ROW0: track 66.6 -> 115.7 mm, vias 1 -> 2
- net ROW1: track 41.9 -> 90.3 mm, vias 0 -> 2
- net COL2: track 67.7 -> 115.9 mm
- net COL0: track 58.7 -> 106.2 mm
- net COL5: track 117.1 -> 164.6 mm
- net COLB: track 63.0 -> 110.1 mm, vias 0 -> 1
- net COL4: track 123.4 -> 169.9 mm
- net COL1: track 59.4 -> 105.7 mm
- net COLA: track 63.0 -> 108.7 mm, vias 0 -> 1
- net COL9: track 80.4 -> 125.7 mm, vias 0 -> 1
- net COL8: track 96.4 -> 140.1 mm, vias 0 -> 1
- net COL3: track 83.1 -> 126.5 mm
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Other:
- net class +3V3: trace_width 0.508 -> 0.2
- net class Power: trace_width 0.508 -> 0.2

Commit message: Prepared Gerbers
Parts:
- renumbered BOOTSEL1 to BOOTSEL, RUN1 to RUN
Routing:
- net COL7: track 185.4 -> 169.1 mm
- net COL6: track 176.6 -> 173.2 mm
- net COLB: track 110.1 -> 108.6 mm
- net D-: track 30.4 -> 29.5 mm
- net ROW0: track 115.7 -> 114.9 mm
- net +3V3: track 169.7 -> 169.0 mm
- net COLA: track 108.7 -> 108.0 mm
- net GND: track 240.0 -> 240.7 mm
- net ROW3: track 154.5 -> 155.1 mm
- net COL9: track 125.7 -> 125.1 mm
- net +5V: track 37.1 -> 37.0 mm, vias 3 -> 2
- added copper zone on B.Cu, net GND
- added copper zone on F.Cu, net GND
Other:
- board text added: "->|-"

Commit message: Replaced the mini-USB connector with USB-C
Parts:
- removed USB1: Molex-0548190589, random-keyboard-parts:Molex-0548190589
- added G***: LOGO, Silkscreens:Crowfeet75, B.Cu at (145.8, 313.2)
- added G***: LOGO, Silkscreens:Crowfeet75, F.Cu at (144.3, 313.2)
- added G***: LOGO, Silkscreens:Crowfeet75, F.Cu at (145.8, 176.3)
- added G***: LOGO, Silkscreens:Crowfeet75, F.Cu at (149.4, 52.1)
- added J32: USB_C_Receptacle_USB2.0, Connector_USB:USB_C_Receptacle_Palconn_UTC16-G, B.Cu at (147.3, 157.0)
- added R8: 5.1k, Resistor_SMD:R_0805_2012Metric, B.Cu at (145.8, 165.0)
- added R9: 5.1k, Resistor_SMD:R_0805_2012Metric, B.Cu at (150.1, 165.0)
- moved F1 2.44 mm to (143.0, 165.0)
- renumbered BOOTSEL to BOOTSEL1, RUN to RUN1
Routing:
- net GND: track 240.7 -> 265.7 mm, vias 18 -> 19
- net Net-(USB1-Pad6): track 16.3 -> 0.00 mm
- net Net-(F1-Pad2): track 6.22 -> 15.4 mm, vias 0 -> 3
- net Net-(J32-PadB5): track 0.00 -> 7.51 mm
- net D-: track 29.5 -> 34.2 mm
- net Net-(J32-PadA5): track 0.00 -> 4.72 mm
- net D+: track 30.4 -> 33.8 mm
Other:
- net class Power: trace_width 0.2 -> 0.508
- board text added: "Thumbs Up! by Sasha Karmanov October 28, 2022 https://github.com/ak66666/ThumbsUpUnsplitV2Rp2040"
- board text removed: "Thumbs Up! by Sasha Karmanov October 28, 2022 https://github.com/ak66666/ThumbsUpUnsplitV2"

Commit message: Added a missing line SS-N
Parts:
- removed G*** (x4): LOGO, Silkscreens:Crowfeet75
- moved RUN1 0.67 mm to (127.0, 228.8)
- moved BOOTSEL1 0.43 mm to (134.9, 228.8)
Connections:
- IC1 pad 56: Net-(IC1-Pad56) -> QSPI_SSN
- IC2 pad 1: Net-(IC2-Pad1) -> QSPI_SSN
- R3 pad 2: Net-(IC2-Pad1) -> QSPI_SSN
- R7 pad 1: Net-(IC2-Pad1) -> QSPI_SSN
Routing:
- net QSPI_SSN: track 0.00 -> 33.5 mm
- net Net-(IC2-Pad1): track 5.83 -> 0.00 mm
- net QSPI_SD2: track 27.0 -> 26.2 mm
- net Net-(BOOTSEL1-Pad1): track 61.4 -> 62.0 mm
- net QSPI_SD1: track 27.6 -> 27.0 mm
- net Net-(IC1-Pad26): track 27.7 -> 27.2 mm
- net GND: track 265.7 -> 266.2 mm

Commit message: Reviewing USB-C Option before ordering
Parts:
- added G***: LOGO, Silkscreens:Crowfeet75, F.Cu at (146.6, 37.8)
- added G***: LOGO, Silkscreens:Crowfeet75, F.Cu at (145.6, 318.4)
- added G***: LOGO, Silkscreens:Crowfeet75, F.Cu at (145.9, 159.8)
- added G***: LOGO, Silkscreens:Crowfeet75, B.Cu at (146.0, 321.2)

Commit message: Retraced the lower PCB
Parts:
- removed the G*** at (146.6, 37.8)
- removed the G*** at (145.6, 318.4)
- removed the G*** at (145.9, 159.8)
- removed the G*** at (146.0, 321.2)
- added G***: LOGO, Silkscreens:Crowfeet75, B.Cu at (145.9, 313.3)
- added G***: LOGO, Silkscreens:Crowfeet75, F.Cu at (156.8, 323.2)
- added G***: LOGO, Silkscreens:Crowfeet75, F.Cu at (158.2, 165.8)
- added G***: LOGO, Silkscreens:Crowfeet75, F.Cu at (149.2, 31.6)
- added H1: MountingHole_Pad, MountingHole:MountingHole_6.4mm_M6_Pad_Via, F.Cu at (145.1, 343.9)
- added H2: MountingHole_Pad, MountingHole:MountingHole_6.4mm_M6_Pad_Via, F.Cu at (145.1, 326.4)
- added H3: MountingHole_Pad, MountingHole:MountingHole_6.4mm_M6_Pad_Via, F.Cu at (145.1, 308.9)
- moved J1 7.62 mm to (47.9, 326.9), turned to 158 degrees
- moved J28 7.61 mm to (242.7, 326.7), turned to 202 degrees
Connections:
- J11 pad 1: Net-(J11-Pad1) -> GND
- J11 pad 2: Net-(J11-Pad2) -> GND
- J11 pad 3: Net-(J11-Pad3) -> GND
- J11 pad 4: Net-(J11-Pad4) -> GND
- J12 pad 1: Net-(J12-Pad1) -> Net-(H1-Pad1)
- J12 pad 2: Net-(J12-Pad2) -> Net-(H1-Pad1)
- J12 pad 3: Net-(J12-Pad3) -> Net-(H1-Pad1)
- J12 pad 4: Net-(J12-Pad4) -> Net-(H1-Pad1)
- J15 pad 1: Net-(J15-Pad1) -> GND
- J15 pad 2: Net-(J15-Pad2) -> GND
- J15 pad 3: Net-(J15-Pad3) -> GND
- J15 pad 4: Net-(J15-Pad4) -> GND
- J16 pad 1: Net-(J16-Pad1) -> Net-(H1-Pad1)
- J16 pad 2: Net-(J16-Pad2) -> Net-(H1-Pad1)
- J16 pad 3: Net-(J16-Pad3) -> Net-(H1-Pad1)
- J16 pad 4: Net-(J16-Pad4) -> Net-(H1-Pad1)
Routing:
- net GND: track 266.2 -> 332.6 mm
- net COL7: track 169.1 -> 213.1 mm
- net Net-(J1-Pad4): track 130.2 -> 91.1 mm, vias 1 -> 0
- net COL4: track 169.7 -> 206.9 mm
- net Net-(J28-Pad4): track 126.8 -> 94.3 mm, vias 0 -> 1
- net Net-(J1-Pad3): track 107.5 -> 79.2 mm, vias 1 -> 0
- net Net-(J28-Pad1): track 115.7 -> 93.3 mm, vias 1 -> 0
- net Net-(J28-Pad3): track 102.7 -> 80.5 mm, vias 1 -> 0
- net Net-(J28-Pad2): track 95.0 -> 73.6 mm, vias 2 -> 0
- net Net-(J29-Pad4): track 27.4 -> 47.6 mm
- net Net-(J1-Pad2): track 96.8 -> 77.1 mm
- net Net-(J30-Pad4): track 25.9 -> 43.2 mm
- net Net-(J31-Pad4): track 27.6 -> 44.3 mm
- net Net-(J2-Pad2): track 84.9 -> 74.7 mm, vias 0 -> 1
- net Net-(J31-Pad3): track 55.2 -> 65.4 mm, vias 0 -> 1
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- added copper zone on B.Cu, net Net-(H1-Pad1)
