File: ThumbsUp.sch (KiCad schematic (older format))
At the start: 156 parts, among them IC1 RP2040, IC2 W25Q128JVSIM, J1 Conn_01x04_Male, J10 Raiser_Male, J11 Raiser_Female, J12 Raiser_Male, J13 Raiser_Female, J14 Raiser_Male, J15 Raiser_Female, J16 Raiser_Male, J17 Raiser_Female, J18 Raiser_Male, J19 52559-1233, J2 Conn_01x04_Male, J20 Conn_01x04_Female, J21 Conn_01x04_Female, J22 Conn_01x04_Female, J23 Conn_01x04_Female, J24 Conn_01x04_Male, J25 Conn_01x04_Male, J26 Conn_01x04_Male, J27 Conn_01x04_Male, J28 Conn_01x04_Female, J29 Conn_01x04_Female, J3 Conn_01x04_Female, J30 Conn_01x04_Female, J31 Conn_01x04_Female, J32 USB_C_Receptacle_USB2.0, J33 STX-3501-3N, J4 Conn_01x04_Male, J5 Conn_01x04_Female, J6 Conn_01x04_Male, J7 Conn_01x04_Male, J8 Conn_01x04_Male, J9 Raiser_Female, U1 NCP1117-3.3_SOT223, Y1 ABLS-12.000MHZ-B4-T

Commit message: Modified schematics: added third thumb button, replaced pushbuttons with through-hole ones
Parts:
- removed BOOTSEL1, RUN1: TL1016AAF220QG, TL1016AAF220QG:TL1016AAF220QG, symbol TL1016AAF220QG:TL1016AAF220QG
- removed J33: STX-3501-3N, STX-3501-3N:STX35013N, symbol STX-3501-3N:STX-3501-3N
- added BOOTSEL1, RUN1: BUTT-4, BUTT-4:BUTT4, symbol BUTT-4:BUTT-4
- added D45, D46: D_Small, Diode_SMD:D_SOD-123, symbol Device:D_Small
- added MX45: SwLThumb3, keyswitches:Kailh_socket_PG1350_optional, symbol ThumbsUp-rescue:MX-NoLED-MX_Alps_Hybrid
- added MX46: SwRThumb3, keyswitches:Kailh_socket_PG1350_optional, symbol ThumbsUp-rescue:MX-NoLED-MX_Alps_Hybrid
- R7: value DNF -> 10K
Connections:
- wire segments 501 -> 525
- no-connect marks 30 -> 22
Other:
- moved on the sheet: J13, J14
